File: PCB/PPU_LITE.sch (EAGLE design)
At the start: 86 parts, among them CON1 DIP40, J1 NTSC/PAL, J2 DENDY, J3 PALSEL0, J4 PALSEL1, J9 BYPASS, T1 BC847, U1 EP1C3T100C8N, U2 EPCS4, U3 SN74LVC8T245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

Commit message: Add files via upload
Parts:
- removed C5: 22uF, rcl_my:C-EUC0603
- added R28, R29, R30: 1k, rcl:R-EU_R0805
- added R31: 100k, rcl:R-EU_R0805
Connections:
- net +3V3: now also R29.1, R30.1; no longer C5.2
- net GND: now also R28.1, R31.2
- net N$13: now also R31.1
- net TCK: now also R28.2
- net TDI: now also R29.2
- net TMS: now also R30.2
Other:
- moved on the sheet: X1-1, X1-10, X1-2, X1-3, X1-4, X1-5, X1-6, X1-7, X1-8, X1-9

Commit message: Add files via upload
Parts:
- added J5, J6: PIN1-2, con-faston:PIN1-2
- L1: value (none) -> BLM31
Connections:
- net VRAMA10: now also J6.1
- net VRAMCS: now also J5.1
Changed lines of the file:
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@@
 <part name="C9" library="rcl_my" deviceset="C-EU" device="C0603" package3d_urn="urn:adsk.eagle:package:23616/2" value="0.1uF"/>
 <part name="JP2" library="pinhead" library_urn="urn:adsk.eagle:library:325" deviceset="PINHD-1X9" device="" package3d_urn="urn:adsk.eagle:package:22483/2"/>
-<part name="L1" library="rcl_my" deviceset="L-EU" device="L0201" package3d_urn="urn:adsk.eagle:package:23513/2"/>
+<part name="L1" library="rcl_my" deviceset="L-EU" device="L0201" package3d_urn="urn:adsk.eagle:package:23513/2" value="BLM31"/>
 <part name="C21" library="rcl_my" deviceset="C-EU" device="C0603" package3d_urn="urn:adsk.eagle:package:23616/2" value="0.1uF"/>
 <part name="GND47" library="supply1" library_urn="urn:adsk.eagle:library:371" deviceset="GND" device=""/>
@@
 <part name="R31" library="rcl" library_urn="urn:adsk.eagle:library:334" deviceset="R-EU_" device="R0805" package3d_urn="urn:adsk.eagle:package:23553/2" value="100k"/>
 <part name="GND20" library="supply1" library_urn="urn:adsk.eagle:library:371" deviceset="GND" device=""/>
+<part name="J5" library="con-faston" library_urn="urn:adsk.eagle:library:144" deviceset="PIN1-2" device="" package3d_urn="urn:adsk.eagle:package:6764/1"/>
+<part name="J6" library="con-faston" library_urn="urn:adsk.eagle:library:144" deviceset="PIN1-2" device="" package3d_urn="urn:adsk.eagle:package:6764/1"/>
 </parts>
 <sheets>
@@
 </instance>
 <instance part="L1" gate="G$1" x="-88.9" y="-7.62" smashed="yes" rot="R90">
-<attribute name="NAME" x="-87.63" y="-4.0386" size="1.778" layer="95" rot="R180"/>
+<attribute name="NAME" x="-87.63" y="-1.4986" size="1.778" layer="95" rot="R180"/>
 <attribute name="VALUE" x="-85.09" y="-4.318" size="1.778" layer="96" rot="R180"/>
 </instance>
@@
 <instance part="GND20" gate="1" x="-83.82" y="93.98" smashed="yes" rot="R180">
 <attribute name="VALUE" x="-81.28" y="96.52" size="1.778" layer="96" rot="R180"/>
+</instance>
+<instance part="J5" gate="G$1" x="-193.04" y="114.3" smashed="yes" rot="MR0">
+<attribute name="NAME" x="-190.5" y="115.57" size="1.778" layer="95" rot="MR0"/>
+<attribute name="VALUE" x="-190.5" y="111.76" size="1.778" layer="96" rot="MR0"/>
+</instance>
+<instance part="J6" gate="G$1" x="-193.04" y="99.06" smashed="yes" rot="MR0">
+<attribute name="NAME" x="-190.5" y="100.33" size="1.778" layer="95" rot="MR0"/>
+<attribute name="VALUE" x="-190.5" y="96.52" size="1.778" layer="96" rot="MR0"/>
 </instance>
 </instances>
@@
 <segment>
 <pinref part="U5" gate="G$1" pin="A1"/>
-<wire x1="-162.56" y1="114.3" x2="-175.26" y2="114.3" width="0.1524" layer="91"/>
 <label x="-175.26" y="114.3" size="1.778" layer="95"/>
+<pinref part="J5" gate="G$1" pin="1"/>
+<wire x1="-162.56" y1="114.3" x2="-187.96" y2="114.3" width="0.1524" layer="91"/>
 </segment>
 </net>
@@
 <segment>
 <pinref part="U5" gate="G$1" pin="A7"/>
-<wire x1="-162.56" y1="99.06" x2="-175.26" y2="99.06" width="0.1524" layer="91"/>
 <label x="-175.26" y="99.06" size="1.778" layer="95"/>
-</segment>
-</net>
+<pinref part="J6" gate="G$1" pin="1"/>
+<wire x1="-162.56" y1="99.06" x2="-187.96" y2="99.06" width="0.1524" layer="91"/>
+</segment>
+</net>
