File: PCB Lattice/V3/PPU_LITE_LATT_V3.sch (EAGLE design)
At the start: 93 parts, among them CON1 DIP40, J1 NTSC/PAL, J2 DENDY, J3 PALSEL0, J4 PALSEL1, J5 PALSEL2, J9 BYPASS, T1 BC847, U1 LCMXO2-1200HC, U2 LS245NSR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

Commit message: Add files via upload
Connections:
- net GND: now also U1.GND@8; no longer CON1.EXT0, CON1.EXT1, U1.GNG@8
Changed lines of the file:
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@@
 <pinref part="GND29" gate="1" pin="GND"/>
 <wire x1="-68.58" y1="73.66" x2="-68.58" y2="71.12" width="0.1524" layer="91"/>
-<pinref part="CON1" gate="G$1" pin="EXT0"/>
-<wire x1="-66.04" y1="88.9" x2="-68.58" y2="88.9" width="0.1524" layer="91"/>
-<wire x1="-68.58" y1="88.9" x2="-68.58" y2="86.36" width="0.1524" layer="91"/>
 <junction x="-68.58" y="73.66"/>
-<pinref part="CON1" gate="G$1" pin="EXT1"/>
-<wire x1="-68.58" y1="86.36" x2="-68.58" y2="83.82" width="0.1524" layer="91"/>
 <wire x1="-68.58" y1="83.82" x2="-68.58" y2="81.28" width="0.1524" layer="91"/>
 <wire x1="-68.58" y1="81.28" x2="-68.58" y2="73.66" width="0.1524" layer="91"/>
-<wire x1="-66.04" y1="86.36" x2="-68.58" y2="86.36" width="0.1524" layer="91"/>
-<junction x="-68.58" y="86.36"/>
-<pinref part="CON1" gate="G$1" pin="EXT2"/>
-<wire x1="-66.04" y1="83.82" x2="-68.58" y2="83.82" width="0.1524" layer="91"/>
-<junction x="-68.58" y="83.82"/>
 <pinref part="CON1" gate="G$1" pin="EXT3"/>
 <wire x1="-66.04" y1="81.28" x2="-68.58" y2="81.28" width="0.1524" layer="91"/>
 <junction x="-68.58" y="81.28"/>
+<pinref part="CON1" gate="G$1" pin="EXT2"/>
+<wire x1="-66.04" y1="83.82" x2="-68.58" y2="83.82" width="0.1524" layer="91"/>
 </segment>
 <segment>
@@
 <wire x1="-2.54" y1="33.02" x2="-2.54" y2="40.64" width="0.1524" layer="91"/>
 <junction x="-2.54" y="40.64"/>
-<pinref part="U1" gate="G$1" pin="GNG@8"/>
+<pinref part="U1" gate="G$1" pin="GND@8"/>
 </segment>
 <segment>
