File: PCB Lattice/V3/PPU_LITE_LATT_V3.sch (EAGLE design)
At the start: 93 parts, among them CON1 DIP40, J1 NTSC/PAL, J2 DENDY, J3 PALSEL0, J4 PALSEL1, J5 PALSEL2, J9 BYPASS, T1 BC847, U1 LCMXO2-1200HC, U2 LS245NSR, U3 SN74LVC8T245, U4 SN74LVC8T245, U5 SN74LVC541A, U6 SN74LVC1G17DBVR, U7 THS7374IPWR, X1 057-010-1

Commit message: Add files via upload
Parts:
- renumbered R10 to R35, R11 to R36, R9 to R34, RN1 to RN16, RN2 to RN15, RN3 to RN17
Connections:
- removed net +3V3: C11.2, C13.1, C14.2, C15.2, C16.2, C17.2, C18.1, C19.2, C20.1, C21.1, C4.2, C5.2, C8.2, C9.1, D1.A, R2.2, R6.2, U1.VCC_INT@2, U1.VCC_IO0@1, U1.VCC_IO0@2, U1.VCC_IO1@1, U1.VCC_IO1@2, U1.VCC_IO2@1, U1.VCC_IO3@1, U1.VCC_IO3@2, U1.VCC_IO3@3, U3.VCCB@1, U3.VCCB@2, U4.VCCA, U5.VCC, U6.VCC, VR1.VOUT
- removed net N$39: C23.1, U1.VCC_INT@1, U1.VCC_IO2@2
- removed net N$46: RN16A.2, RN16B.2, RN16C.2
- removed net N$47: RN16A.1, RN16B.1, RN16D.2, RN17A.2
- new net N$48: RN16A.1, RN16B.1, RN16C.2
- new net N$57: RN16A.2, RN16B.2, RN16D.2, RN17A.2
- new net VCCIO: C11.2, C13.1, C14.2, C15.2, C16.2, C17.2, C18.1, C19.2, C20.1, C21.1, C23.1, C4.2, C5.2, C8.2, C9.1, D1.A, R2.2, R6.2, U1.VCC_INT@1, U1.VCC_INT@2, U1.VCC_IO0@1, U1.VCC_IO0@2, U1.VCC_IO1@1, U1.VCC_IO1@2, U1.VCC_IO2@1, U1.VCC_IO2@2, U1.VCC_IO3@1, U1.VCC_IO3@2, U1.VCC_IO3@3, U3.VCCB@1, U3.VCCB@2, U4.VCCA, U5.VCC, U6.VCC, VR1.VOUT
- net +5V: now also U2.DIR
- net GND: now also C21.2, C22.1
- net N$21: now also RN7A.1, RN7B.1; no longer RN7A.2, RN7B.2
- net N$22: now also RN7A.2, RN7B.2; no longer RN7A.1, RN7B.1
- net N$32: now also RN4A.1, RN4B.1; no longer RN4A.2, RN4B.2
- net N$33: now also RN4A.2, RN4B.2; no longer RN4A.1, RN4B.1
Other:
- moved on the sheet: C22

Commit message: Add files via upload
Parts:
- removed RN14, RN15: 2k, resistor-dil:4R-N0603-ARC
- removed RN17: 1k, resistor-dil:4R-N0603-ARC
- added JP3: VRAMCS, pinhead:PINHD-1X1
- added JP4: VRAMA10, pinhead:PINHD-1X1
- added RN1, RN2: 51, resistor-dil:4R-N0603-ARC
- added RN3: 2k, resistor-dil:4R-N0603-ARC
- JP1: value (none) -> CO/CS
- LED1: value (none) -> GNL-1206YC
- RN10: value 51 -> 1k
- RN11: value 51 -> 2k
- RN5: value 2k -> 1k
- RN6: value 1k -> 2k
Connections:
- removed net N$17: RN8A.2, RN9A.1, RN9B.2
- removed net N$32: RN4A.1, RN4B.1, RN4C.2
- removed net N$33: RN4A.2, RN4B.2, RN4D.2, RN6A.2
- removed net N$36: RN5B.2, RN6B.1, RN6C.2
- removed net N$37: RN5C.2, RN6C.1, RN6D.2
- removed net N$57: RN16A.2, RN16B.2, RN16D.2, RN17A.2
- removed net VRAMA10: U5.A7
- removed net VRAMCS: U5.A8
- new net N$3: JP4.1, U5.A7
- new net N$39: JP3.1, U5.A8
- new net N$41: RN16B.1, RN16C.2, RN16D.2
- new net N$45: RN10D.1, RN16A.1, RN16C.1, RN16D.1
- new net N$46: RN12D.1, RN13C.1, RN13D.2
- new net N$47: RN12C.1, RN13B.1, RN13C.2
- new net N$50: RN11B.1, RN11C.2, RN11D.2
- new net N$51: RN11A.1, RN11C.1, RN11D.1, RN13D.1
- net /DBE_FPGA: now also U1.IO21_CSS; no longer U1.IO21
- net /PRD_FPGA: now also RN2C.1; no longer RN11C.1
- net /PWR_FPGA: now also RN2D.1; no longer RN11D.1
- net A2_FPGA: now also U1.IO9_PCLKT3_1; no longer U1.IO9
- net B0: now also RN7B.2; no longer RN7C.1
- net B1: now also RN7A.2; no longer RN7D.1
- net B2: now also RN8D.2; no longer RN8A.1
- net B3: now also RN8C.2; no longer RN8B.1
- net B4: now also RN8B.2; no longer RN8C.1
- net B5: now also RN8A.2; no longer RN8D.1
- net CLK_FPGA: now also U1.IO27_PCLKT2_0; no longer U1.IO27
- net COMP0: now also RN3C.2; no longer RN14B.1
- net COMP1: now also RN3B.2; no longer RN14C.1
- net COMP2: now also RN3A.2, U1.JTAGENB_IO66; no longer RN14D.1, U1.IO66
- net COMP3: now also RN4D.2, U1.PROGRAMN_IO65; no longer RN12A.1, U1.IO65
- net COMP4: now also RN4C.2; no longer RN12B.1
- net COMP5: now also RN4B.2, U1.INITN_IO63; no longer RN12C.1, U1.IO63
- net COMP6: now also RN4A.2, U1.DONE_IO62; no longer RN12D.1, U1.IO62
- net CS_FPGA: now also U1.IO40_SI_SPISI; no longer U1.IO40
- net DB1_FPGA: now also U1.IO18_PCLKC3_0; no longer U1.IO18
- net DB2_FPGA: now also U1.IO17_PCLKT3_0; no longer U1.IO17
- net DENDY: now also U1.SDA_PCLKC0_0_IO69; no longer U1.IO69
- net G0: now also RN11B.2; no longer RN4C.1
- net G1: now also RN11A.2; no longer RN4D.1
- net G2: now also RN12D.2; no longer RN5A.1
- net G3: now also RN12C.2, U1.PCLKT1_0_IO51; no longer RN5B.1, U1.IO51
- net G4: now also RN12B.2, U1.PCLKC1_0_IO50; no longer RN5C.1, U1.IO50
- net G5: now also RN12A.2; no longer RN5D.1
- net GND: now also C1.1, C10.1, C11.1, C12.2, C13.2, C17.1, C2.-, C24.1, C25.1, C3.1, C4.1, C5.1, C6.2, C7.2, C8.1, C9.2, RN3D.2, U1.GNG@8, VR1.GND, X1-8.S; no longer RN14A.1, U1.GND@8, X1-2.S
- net HS_FPGA: now also U1.IO39_SN; no longer U1.IO39
- net N$10: now also RN2D.2; no longer RN11D.2
- net N$11: now also RN2C.2; no longer RN11C.2
- net N$12: now also RN2B.2; no longer RN11B.2
- net N$13: now also RN2A.2; no longer RN11A.2
- net N$16: now also RN1D.2; no longer RN10D.2
- net N$18: now also RN1C.2; no longer RN10C.2
- net N$19: now also RN1B.2; no longer RN10B.2
- net N$20: now also RN1A.2; no longer RN10A.2
- net N$21: now also RN8D.1, RN9C.1, RN9D.2; no longer RN7A.1, RN7B.1, RN7C.2
- net N$22: now also RN8C.1, RN9B.1, RN9C.2; no longer RN7A.2, RN7B.2, RN7D.2, RN9A.2
- net N$23: now also RN8B.1, RN9A.1, RN9B.2; no longer RN8B.2, RN9B.1, RN9C.2
- net N$26: now also RN3C.1, RN3D.1; no longer RN14A.2, RN14B.2
- net N$27: now also RN7B.1, RN7C.2, RN7D.2; no longer RN8C.2, RN9C.1, RN9D.2
- net N$28: now also RN3B.1; no longer RN14C.2
- net N$29: now also RN8A.1, RN9A.2; no longer RN8D.2, RN9D.1
- net N$31: now also RN7A.1, RN7C.1, RN7D.1, RN9D.1; no longer RN5A.2, RN6A.1, RN6B.2
- net N$34: now also RN4A.1, RN5A.2; no longer RN12D.2, RN13D.1
- net N$38: now also RN12A.1, RN13A.2; no longer RN5D.2, RN6D.1
- net N$43: now also RN10C.1, RN10D.2, RN6D.1; no longer RN15A.2, RN17A.1, RN17B.2
- net N$48: now also RN12B.1, RN13A.1, RN13B.2; no longer RN16A.1, RN16B.1, RN16C.2
- net N$53: now also RN10B.1, RN10C.2, RN6C.1; no longer RN15B.2, RN17B.1, RN17C.2
- net N$54: now also RN10A.1, RN10B.2, RN6B.1; no longer RN15C.2, RN17C.1, RN17D.2
- net N$55: now also RN10A.2, RN6A.1; no longer RN15D.2, RN17D.1
- net N$6: now also RN4D.1, RN5C.1, RN5D.2; no longer RN12A.2, RN13A.1, RN13B.2
- net N$7: now also RN3A.1, RN5D.1; no longer RN13A.2, RN14D.2
- net N$8: now also RN4C.1, RN5B.1, RN5C.2; no longer RN12B.2, RN13B.1, RN13C.2
- net N$9: now also RN4B.1, RN5A.1, RN5B.2; no longer RN12C.2, RN13C.1, RN13D.2
- net PA10_FPGA: now also RN1C.1, U1.IO4_PCLKC3_2; no longer RN10C.1, U1.IO4
- net PA11_FPGA: now also RN1D.1, U1.IO3_PCLKT3_2; no longer RN10D.1, U1.IO3
- net PA12_FPGA: now also RN2A.1; no longer RN11A.1
- net PA13_FPGA: now also RN2B.1; no longer RN11B.1
- net PA8_FPGA: now also RN1A.1; no longer RN10A.1
- net PA9_FPGA: now also RN1B.1; no longer RN10B.1
- net PALSEL0: now also U1.SCL_PCLKT0_0_IO70; no longer U1.IO70
- net PALSEL1: now also U1.PCLKC0_1_IO71; no longer U1.IO71
- net PALSEL2: now also U1.PCLKT0_1_IO72; no longer U1.IO72
- net PD4_FPGA: now also U1.IO32_PCLKC2_1; no longer U1.IO32
- net PD5_FPGA: now also U1.IO31_PCLKT2_1; no longer U1.IO31
- net PD_DIR: now also U1.IO28_PCLKC2_0; no longer U1.IO28
- net R0: now also RN16B.2; no longer RN16C.1
- net R1: now also RN16A.2; no longer RN16D.1
- net R2: now also RN6D.2; no longer RN15A.1
- net R3: now also RN6C.2; no longer RN15B.1
- net R4: now also RN6B.2; no longer RN15C.1
- net R5: now also RN6A.2; no longer RN15D.1
- net VR10_FPGA: now also U1.IO10_PCLKC3_1; no longer U1.IO10
Other:
- moved on the sheet: C24, C25, J9, JP1, JP2, LED1, R12, R13, R14, R15, R16, R17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

Commit message: Add files via upload
Parts:
- JP2: value (none) -> AVOUT
Other:
- moved on the sheet: C10, C7, C8, C9, RN1A, RN1B, RN1C, RN1D, RN2A, RN2B, RN2C, RN2D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

Commit message: Add files via upload
Parts:
- removed RN16: 2k, resistor-dil:4R-N0603-ARC
- added RN14: 1k, resistor-dil:4R-N0603-ARC
- RN10, RN13, RN9: value 1k -> 2k
- RN11, RN8: value 2k -> 1k
Connections:
- net +5V: now also C10.1; no longer C10.2
- net B0: now also RN12B.2; no longer RN7B.2
- net B1: now also RN12A.2; no longer RN7A.2
- net B2: now also RN13D.2; no longer RN8D.2
- net B3: now also RN13C.2; no longer RN8C.2
- net B4: now also RN13B.2; no longer RN8B.2
- net B5: now also RN13A.2; no longer RN8A.2
- net G0: now also RN9B.2; no longer RN11B.2
- net G1: now also RN9A.2; no longer RN11A.2
- net G2: now also RN10D.2; no longer RN12D.2
- net G3: now also RN10C.2; no longer RN12C.2
- net G4: now also RN10B.2; no longer RN12B.2
- net G5: now also RN10A.2; no longer RN12A.2
- net GND: now also C10.2, C8.2; no longer C10.1, C8.1
- net N$21: now also RN13D.1, RN14C.1, RN14D.2; no longer RN8D.1, RN9C.1, RN9D.2
- net N$22: now also RN13C.1, RN14B.1, RN14C.2; no longer RN8C.1, RN9B.1, RN9C.2
- net N$23: now also RN13B.1, RN14A.1, RN14B.2; no longer RN8B.1, RN9A.1, RN9B.2
- net N$27: now also RN12B.1, RN12C.2, RN12D.2; no longer RN7B.1, RN7C.2, RN7D.2
- net N$29: now also RN13A.1, RN14A.2; no longer RN8A.1, RN9A.2
- net N$31: now also RN12A.1, RN12C.1, RN12D.1, RN14D.1; no longer RN7A.1, RN7C.1, RN7D.1, RN9D.1
- net N$38: now also RN10A.1, RN11A.2; no longer RN12A.1, RN13A.2
- net N$41: now also RN6B.1, RN6C.2, RN6D.2; no longer RN16B.1, RN16C.2, RN16D.2
- net N$43: now also RN7D.1, RN8C.1, RN8D.2; no longer RN10C.1, RN10D.2, RN6D.1
- net N$45: now also RN6A.1, RN6C.1, RN6D.1, RN8D.1; no longer RN10D.1, RN16A.1, RN16C.1, RN16D.1
- net N$46: now also RN10D.1, RN11C.1, RN11D.2; no longer RN12D.1, RN13C.1, RN13D.2
- net N$47: now also RN10C.1, RN11B.1, RN11C.2; no longer RN12C.1, RN13B.1, RN13C.2
- net N$48: now also RN10B.1, RN11A.1, RN11B.2; no longer RN12B.1, RN13A.1, RN13B.2
- net N$50: now also RN9B.1, RN9C.2, RN9D.2; no longer RN11B.1, RN11C.2, RN11D.2
- net N$51: now also RN9A.1, RN9C.1, RN9D.1; no longer RN11A.1, RN11C.1, RN13D.1
- net N$53: now also RN7C.1, RN8B.1, RN8C.2; no longer RN10B.1, RN10C.2, RN6C.1
- net N$54: now also RN7B.1, RN8A.1, RN8B.2; no longer RN10A.1, RN10B.2, RN6B.1
- net N$55: now also RN7A.1, RN8A.2; no longer RN10A.2, RN6A.1
- net R0: now also RN6B.2; no longer RN16B.2
- net R1: now also RN6A.2; no longer RN16A.2
- net R2: now also RN7D.2; no longer RN6D.2
- net R3: now also RN7C.2; no longer RN6C.2
- net R4: now also RN7B.2; no longer RN6B.2
- net R5: now also RN7A.2; no longer RN6A.2
- net VCCIO: now also C8.1; no longer C8.2
Other:
- moved on the sheet: C1, C10, C2, C3, C6, C7, C8, C9, RN10A, RN10B, RN10C, RN10D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

Commit message: Add files via upload
Connections:
- net GND: now also U1.GND@8; no longer U1.GNG@8
Other:
- moved on the sheet: C4, C5
Changed lines of the file:
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@@
 <attribute name="VALUE" x="-169.418" y="124.841" size="1.778" layer="96"/>
 </instance>
-<instance part="C4" gate="G$1" x="-127" y="114.3" smashed="yes" rot="R180">
-<attribute name="NAME" x="-125.73" y="129.159" size="1.778" layer="95" rot="R180"/>
-<attribute name="VALUE" x="-122.936" y="126.619" size="1.778" layer="96" rot="R180"/>
+<instance part="C4" gate="G$1" x="-127" y="111.76" smashed="yes" rot="R180">
+<attribute name="NAME" x="-125.73" y="126.619" size="1.778" layer="95" rot="R180"/>
+<attribute name="VALUE" x="-122.936" y="124.079" size="1.778" layer="96" rot="R180"/>
 </instance>
 <instance part="C7" gate="G$1" x="-190.5" y="12.7" smashed="yes" rot="R180">
@@
 <attribute name="VALUE" x="-116.84" y="104.14" size="1.778" layer="96"/>
 </instance>
-<instance part="C5" gate="G$1" x="-114.3" y="114.3" smashed="yes" rot="R180">
-<attribute name="NAME" x="-113.03" y="129.159" size="1.778" layer="95" rot="R180"/>
-<attribute name="VALUE" x="-111.252" y="126.619" size="1.778" layer="96" rot="R180"/>
+<instance part="C5" gate="G$1" x="-114.3" y="111.76" smashed="yes" rot="R180">
+<attribute name="NAME" x="-113.03" y="126.619" size="1.778" layer="95" rot="R180"/>
+<attribute name="VALUE" x="-111.252" y="124.079" size="1.778" layer="96" rot="R180"/>
 </instance>
 <instance part="LED1" gate="G$1" x="228.6" y="-175.26" smashed="yes">
@@
 <wire x1="-2.54" y1="33.02" x2="-2.54" y2="40.64" width="0.1524" layer="91"/>
 <junction x="-2.54" y="40.64"/>
-<pinref part="U1" gate="G$1" pin="GNG@8"/>
+<pinref part="U1" gate="G$1" pin="GND@8"/>
 </segment>
 <segment>
@@
 </segment>
 <segment>
-<pinref part="GND39" gate="1" pin="GND"/>
-<pinref part="C4" gate="G$1" pin="1"/>
-<wire x1="-127" y1="109.22" x2="-127" y2="111.76" width="0.1524" layer="91"/>
-</segment>
-<segment>
-<pinref part="GND44" gate="1" pin="GND"/>
-<pinref part="C5" gate="G$1" pin="1"/>
-<wire x1="-114.3" y1="109.22" x2="-114.3" y2="111.76" width="0.1524" layer="91"/>
-</segment>
-<segment>
 <pinref part="C12" gate="G$1" pin="2"/>
 <pinref part="GND47" gate="1" pin="GND"/>
@@
 <pinref part="GND28" gate="1" pin="GND"/>
 </segment>
+<segment>
+<pinref part="GND44" gate="1" pin="GND"/>
+<pinref part="C5" gate="G$1" pin="1"/>
+</segment>
+<segment>
+<pinref part="GND39" gate="1" pin="GND"/>
+<pinref part="C4" gate="G$1" pin="1"/>
+</segment>
 </net>
 <net name="TDI" class="0">
@@
 </segment>
 <segment>
+<pinref part="U4" gate="G$1" pin="VCCA"/>
+<pinref part="VCC10" gate="G$1" pin="VCCIO"/>
+<wire x1="-165.1" y1="-60.96" x2="-190.5" y2="-60.96" width="0.1524" layer="91"/>
+<pinref part="C9" gate="G$1" pin="1"/>
+<wire x1="-190.5" y1="-60.96" x2="-193.04" y2="-60.96" width="0.1524" layer="91"/>
+<wire x1="-190.5" y1="-58.42" x2="-190.5" y2="-60.96" width="0.1524" layer="91"/>
+<junction x="-190.5" y="-60.96"/>
+</segment>
+<segment>
 <pinref part="VCC8" gate="G$1" pin="VCCIO"/>
 <pinref part="VR1" gate="G$1" pin="VOUT"/>
@@
 <wire x1="-114.3" y1="121.92" x2="-127" y2="121.92" width="0.1524" layer="91"/>
 <wire x1="-127" y1="121.92" x2="-132.08" y2="121.92" width="0.1524" layer="91"/>
+<wire x1="-127" y1="119.38" x2="-127" y2="121.92" width="0.1524" layer="91"/>
 <junction x="-127" y="121.92"/>
 <pinref part="C5" gate="G$1" pin="2"/>
+<wire x1="-114.3" y1="119.38" x2="-114.3" y2="121.92" width="0.1524" layer="91"/>
 <junction x="-114.3" y="121.92"/>
 </segment>
-<segment>
-<pinref part="U4" gate="G$1" pin="VCCA"/>
-<pinref part="VCC10" gate="G$1" pin="VCCIO"/>
-<wire x1="-165.1" y1="-60.96" x2="-190.5" y2="-60.96" width="0.1524" layer="91"/>
-<pinref part="C9" gate="G$1" pin="1"/>
-<wire x1="-190.5" y1="-60.96" x2="-193.04" y2="-60.96" width="0.1524" layer="91"/>
-<wire x1="-190.5" y1="-58.42" x2="-190.5" y2="-60.96" width="0.1524" layer="91"/>
-<junction x="-190.5" y="-60.96"/>
-</segment>
 </net>
