File: PPU_MINI/PCB/PPU_MINI.sch (EAGLE design)
At the start: 92 parts, among them CON1 DIP40, J1 NTSC/PAL, J2 DENDY, J3 PALSEL0, J4 PALSEL1, J5 PALSEL2, J9 BYPASS, T1 BC847, U1 LCMXO2-1200HC, U2 BH7240AKV, U3 SN74LVC8T245, U4 SN74LVC8T245, U5 SN74LVC541A, U6 SN74LVC1G17DBVR, U7 THS7374IPWR, X1 057-010-1

Commit message: Add files via upload
Connections:
- net GND: now also X1-8.S; no longer X1-2.S
Other:
- moved on the sheet: X1-1, X1-3, X1-5, X1-7, X1-9
Changed lines of the file:
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@@
 <part name="GND34" library="supply1" library_urn="urn:adsk.eagle:library:371" deviceset="GND" device=""/>
 <part name="X1" library="con-panduit" library_urn="urn:adsk.eagle:library:169" deviceset="057-010-" device="1" package3d_urn="urn:adsk.eagle:package:9203/1"/>
-<part name="GND43" library="supply1" library_urn="urn:adsk.eagle:library:371" deviceset="GND" device=""/>
 <part name="U3" library="SnapEDA-Library" deviceset="SN74LVC8T245" device=""/>
 <part name="U4" library="SnapEDA-Library" deviceset="SN74LVC8T245" device=""/>
@@
 <part name="VCC2" library="supply1" library_urn="urn:adsk.eagle:library:371" deviceset="VCCIO" device=""/>
 <part name="VCC3" library="supply1" library_urn="urn:adsk.eagle:library:371" deviceset="VCCIO" device=""/>
-<part name="VCC4" library="supply1" library_urn="urn:adsk.eagle:library:371" deviceset="VCCIO" device=""/>
 <part name="VCC5" library="supply1" library_urn="urn:adsk.eagle:library:371" deviceset="VCCIO" device=""/>
 <part name="VCC6" library="supply1" library_urn="urn:adsk.eagle:library:371" deviceset="VCCIO" device=""/>
@@
 <part name="C9" library="rcl_my" deviceset="C-EU" device="C0603" package3d_urn="urn:adsk.eagle:package:23616/2" value="0.1uF"/>
 <part name="C10" library="rcl_my" deviceset="C-EU" device="C0603" package3d_urn="urn:adsk.eagle:package:23616/2" value="0.1uF"/>
+<part name="GND43" library="supply1" library_urn="urn:adsk.eagle:library:371" deviceset="GND" device=""/>
+<part name="GND25" library="supply1" library_urn="urn:adsk.eagle:library:371" deviceset="GND" device=""/>
+<part name="VCC4" library="supply1" library_urn="urn:adsk.eagle:library:371" deviceset="VCCIO" device=""/>
 </parts>
 <sheets>
@@
 <attribute name="VALUE" x="-172.72" y="114.3" size="1.778" layer="96"/>
 </instance>
-<instance part="X1" gate="-1" x="129.54" y="-111.76" smashed="yes">
-<attribute name="NAME" x="130.556" y="-112.522" size="1.524" layer="95"/>
-<attribute name="VALUE" x="127" y="-109.855" size="1.778" layer="96"/>
+<instance part="X1" gate="-1" x="121.92" y="-111.76" smashed="yes">
+<attribute name="NAME" x="122.936" y="-112.522" size="1.524" layer="95"/>
+<attribute name="VALUE" x="119.38" y="-109.855" size="1.778" layer="96"/>
 </instance>
 <instance part="X1" gate="-2" x="152.4" y="-111.76" smashed="yes">
 <attribute name="NAME" x="153.416" y="-112.522" size="1.524" layer="95"/>
 </instance>
-<instance part="X1" gate="-3" x="129.54" y="-116.84" smashed="yes">
-<attribute name="NAME" x="130.556" y="-117.602" size="1.524" layer="95"/>
+<instance part="X1" gate="-3" x="121.92" y="-116.84" smashed="yes">
+<attribute name="NAME" x="122.936" y="-117.602" size="1.524" layer="95"/>
 </instance>
 <instance part="X1" gate="-4" x="152.4" y="-116.84" smashed="yes">
 <attribute name="NAME" x="153.416" y="-117.602" size="1.524" layer="95"/>
 </instance>
-<instance part="X1" gate="-5" x="129.54" y="-121.92" smashed="yes">
-<attribute name="NAME" x="130.556" y="-122.682" size="1.524" layer="95"/>
+<instance part="X1" gate="-5" x="121.92" y="-121.92" smashed="yes">
+<attribute name="NAME" x="122.936" y="-122.682" size="1.524" layer="95"/>
 </instance>
 <instance part="X1" gate="-6" x="152.4" y="-121.92" smashed="yes">
 <attribute name="NAME" x="153.416" y="-122.682" size="1.524" layer="95"/>
 </instance>
-<instance part="X1" gate="-7" x="129.54" y="-127" smashed="yes">
-<attribute name="NAME" x="130.556" y="-127.762" size="1.524" layer="95"/>
+<instance part="X1" gate="-7" x="121.92" y="-127" smashed="yes">
+<attribute name="NAME" x="122.936" y="-127.762" size="1.524" layer="95"/>
 </instance>
 <instance part="X1" gate="-8" x="152.4" y="-127" smashed="yes">
 <attribute name="NAME" x="153.416" y="-127.762" size="1.524" layer="95"/>
 </instance>
-<instance part="X1" gate="-9" x="129.54" y="-132.08" smashed="yes">
-<attribute name="NAME" x="130.556" y="-132.842" size="1.524" layer="95"/>
+<instance part="X1" gate="-9" x="121.92" y="-132.08" smashed="yes">
+<attribute name="NAME" x="122.936" y="-132.842" size="1.524" layer="95"/>
 </instance>
 <instance part="X1" gate="-10" x="152.4" y="-132.08" smashed="yes">
 <attribute name="NAME" x="153.416" y="-132.842" size="1.524" layer="95"/>
-</instance>
-<instance part="GND43" gate="1" x="144.78" y="-111.76" smashed="yes" rot="R270">
-<attribute name="VALUE" x="142.24" y="-109.22" size="1.778" layer="96" rot="R270"/>
 </instance>
 <instance part="U3" gate="G$1" x="-147.32" y="-12.7" smashed="yes">
@@
 <attribute name="VALUE" x="-42.418" y="51.562" size="1.778" layer="96" rot="R180"/>
 </instance>
-<instance part="VCC4" gate="G$1" x="144.78" y="-121.92" smashed="yes" rot="R90">
-<attribute name="VALUE" x="145.542" y="-118.618" size="1.778" layer="96" rot="R180"/>
-</instance>
 <instance part="VCC5" gate="G$1" x="-91.44" y="-30.48" smashed="yes" rot="R90">
 <attribute name="VALUE" x="-93.218" y="-29.718" size="1.778" layer="96" rot="R180"/>
@@
 <attribute name="NAME" x="-175.26" y="-60.071" size="1.778" layer="95" rot="R180"/>
 <attribute name="VALUE" x="-172.974" y="-65.151" size="1.778" layer="96" rot="R180"/>
+</instance>
+<instance part="GND43" gate="1" x="144.78" y="-116.84" smashed="yes" rot="R270">
+<attribute name="VALUE" x="142.24" y="-114.3" size="1.778" layer="96" rot="R270"/>
+</instance>
+<instance part="GND25" gate="1" x="144.78" y="-127" smashed="yes" rot="R270">
+<attribute name="VALUE" x="142.24" y="-124.46" size="1.778" layer="96" rot="R270"/>
+</instance>
+<instance part="VCC4" gate="G$1" x="137.16" y="-121.92" smashed="yes" rot="R90">
+<attribute name="VALUE" x="137.922" y="-118.618" size="1.778" layer="96" rot="R180"/>
 </instance>
 </instances>
@@
 <segment>
 <pinref part="X1" gate="-1" pin="S"/>
-<wire x1="124.46" y1="-111.76" x2="116.84" y2="-111.76" width="0.1524" layer="91"/>
-<label x="116.84" y="-111.76" size="1.778" layer="95"/>
+<wire x1="116.84" y1="-111.76" x2="109.22" y2="-111.76" width="0.1524" layer="91"/>
+<label x="109.22" y="-111.76" size="1.778" layer="95"/>
 </segment>
 <segment>
@@
 </net>
 <net name="GND" class="0">
-<segment>
-<pinref part="X1" gate="-2" pin="S"/>
-<pinref part="GND43" gate="1" pin="GND"/>
-<pinref part="X1" gate="-4" pin="S"/>
-<wire x1="147.32" y1="-116.84" x2="147.32" y2="-111.76" width="0.1524" layer="91"/>
-<junction x="147.32" y="-111.76"/>
-</segment>
 <segment>
 <pinref part="GND6" gate="1" pin="GND"/>
@@
 <pinref part="GND38" gate="1" pin="GND"/>
 </segment>
+<segment>
+<pinref part="GND25" gate="1" pin="GND"/>
+<pinref part="X1" gate="-8" pin="S"/>
+</segment>
+<segment>
+<pinref part="X1" gate="-4" pin="S"/>
+<pinref part="GND43" gate="1" pin="GND"/>
+</segment>
 </net>
 <net name="TDI" class="0">
@@
 </segment>
 <segment>
-<wire x1="124.46" y1="-121.92" x2="116.84" y2="-121.92" width="0.1524" layer="91"/>
+<wire x1="116.84" y1="-121.92" x2="109.22" y2="-121.92" width="0.1524" layer="91"/>
 <pinref part="X1" gate="-5" pin="S"/>
-<label x="116.84" y="-121.92" size="1.778" layer="95"/>
+<label x="109.22" y="-121.92" size="1.778" layer="95"/>
 </segment>
 </net>
@@
 </segment>
 <segment>
-<wire x1="124.46" y1="-116.84" x2="116.84" y2="-116.84" width="0.1524" layer="91"/>
+<wire x1="116.84" y1="-116.84" x2="109.22" y2="-116.84" width="0.1524" layer="91"/>
 <pinref part="X1" gate="-3" pin="S"/>
-<label x="116.84" y="-116.84" size="1.778" layer="95"/>
+<label x="109.22" y="-116.84" size="1.778" layer="95"/>
 </segment>
 </net>
@@
 </segment>
 <segment>
-<wire x1="124.46" y1="-127" x2="116.84" y2="-127" width="0.1524" layer="91"/>
+<wire x1="116.84" y1="-127" x2="109.22" y2="-127" width="0.1524" layer="91"/>
 <pinref part="X1" gate="-7" pin="S"/>
-<label x="116.84" y="-127" size="1.778" layer="95"/>
+<label x="109.22" y="-127" size="1.778" layer="95"/>
 </segment>
 </net>
@@
 <pinref part="R21" gate="G$1" pin="1"/>
 <pinref part="C29" gate="G$1" pin="2"/>
-<pinref part="R22" gate="G$1" pin="2"/>
 <pinref part="R22" gate="G$1" pin="2"/>
 <junction x="119.38" y="111.76"/>
@@
 </segment>
 <segment>
+<pinref part="VCC4" gate="G$1" pin="VCCIO"/>
 <pinref part="X1" gate="-6" pin="S"/>
-<pinref part="VCC4" gate="G$1" pin="VCCIO"/>
-</segment>
-</net>
+<wire x1="139.7" y1="-121.92" x2="147.32" y2="-121.92" width="0.1524" layer="91"/>
+</segment>
+</net>

Commit message: Add files via upload
Parts:
- removed C38: 220uF, rcl_my:C-EUC0603
- C12, C25: value 22uF -> 0.1uF
- C28, C6: value 0.1uF -> 22uF
- C33: value 0.1uF -> 0.047uF
- C34: value 0.1uF -> 220uF
- C35: value 22uF -> 27
- C36: value 27 -> 0.1uF
- C37: value 0.047uF -> 0.1uF
- U2: value BH7240AKV -> SN74LVC8T245; device BH7240AKV:BH7240AKV -> SnapEDA-Library:SN74LVC8T245
- U4: value SN74LVC8T245 -> SN74LVC541A; device SnapEDA-Library:SN74LVC8T245 -> SnapEDA-Library:SN74LVC541A
- U5: value SN74LVC541A -> SN74LVC1G17DBVR; device SnapEDA-Library:SN74LVC541A -> SN74LVC1G17DBVR:SN74LVC1G17DBVR
- U6: value SN74LVC1G17DBVR -> THS7374IPWR; device SN74LVC1G17DBVR:SN74LVC1G17DBVR -> THS7374IPWR:THS7374IPWR
- U7: value THS7374IPWR -> BH7240AKV; device THS7374IPWR:THS7374IPWR -> BH7240AKV:BH7240AKV
Connections:
- net +5V: now also C27.2, C28.2, C36.2, C37.2, C6.1, U2.VCCB@1, U2.VCCB@2, U6.VS+, U7.AVCC1, U7.AVCC2, U7.DVDD; no longer C12.1, C24.2, C25.2, C33.2, C34.2, C35.2, U2.AVCC1, U2.AVCC2, U2.DVDD, U4.VCCB@1, U4.VCCB@2, U7.VS+
- net /DBE: now also U4.A1; no longer U5.A1
- net /DBE_FPGA: now also U3./OE, U4.Y1; no longer U4./OE, U5.Y1
- net /PRD: now also U2.DIR; no longer U3.DIR
- net A0: now also U4.A2; no longer U5.A2
- net A0_FPGA: now also U4.Y2; no longer U5.Y2
- net A1: now also U4.A3; no longer U5.A3
- net A1_FPGA: now also U4.Y3; no longer U5.Y3
- net A2: now also U4.A4; no longer U5.A4
- net A2_FPGA: now also U4.Y4; no longer U5.Y4
- net B0: now also U7.B0; no longer U2.B0
- net B1: now also U7.B1; no longer U2.B1
- net B2: now also U7.B2; no longer U2.B2
- net B3: now also U7.B3; no longer U2.B3
- net B4: now also U7.B4; no longer U2.B4
- net B5: now also U7.B5; no longer U2.B5
- net B6: now also U7.B6; no longer U2.B6
- net B7: now also U7.B7; no longer U2.B7
- net BO: now also U7.BOUT; no longer U2.BOUT
- net C: now also C33.1; no longer C37.1
- net CLK: now also U5.A; no longer U6.A
- net DB0: now also U3.B7; no longer U4.B7
- net DB0_FPGA: now also U3.A7; no longer U4.A7
- net DB1: now also U3.B6; no longer U4.B6
- net DB1_FPGA: now also U3.A6; no longer U4.A6
- net DB2: now also U3.B5; no longer U4.B5
- net DB2_FPGA: now also U3.A5; no longer U4.A5
- net DB3: now also U3.B4; no longer U4.B4
- net DB3_FPGA: now also U3.A4; no longer U4.A4
- net DB4: now also U3.B3; no longer U4.B3
- net DB4_FPGA: now also U3.A3; no longer U4.A3
- net DB5: now also U3.B2; no longer U4.B2
- net DB5_FPGA: now also U3.A2; no longer U4.A2
- net DB6: now also U3.B1; no longer U4.B1
- net DB6_FPGA: now also U3.A1; no longer U4.A1
- net DB7: now also U3.B0; no longer U4.B0
- net DB7_FPGA: now also U3.A0; no longer U4.A0
- net G0: now also U7.G0; no longer U2.G0
- net G1: now also U7.G1; no longer U2.G1
- net G2: now also U7.G2; no longer U2.G2
- net G3: now also U7.G3; no longer U2.G3
- net G4: now also U7.G4; no longer U2.G4
- net G5: now also U7.G5; no longer U2.G5
- net G6: now also U7.G6; no longer U2.G6
- net G7: now also U7.G7; no longer U2.G7
- net GND: now also C13.1, C17.2, C18.1, C19.2, C29.1, C30.1, C31.1, C32.1, C37.1, C6.2, U1.GND@8, U2./OE, U2.GND@1, U2.GND@2, U2.GND@3, U4./OE1, U4./OE2, U4.A8, U4.GND, U6.DISABLE, U7.AGND1, U7.AGND2, U7.DGND; no longer C13.2, C17.1, C18.2, C19.1, C23.2, C24.1, C25.1, C26.1, C33.1, C34.1, C6.1, U1.GNG@8, U2.AGND1, U2.AGND2, U2.DGND, U3./OE, U4.GND@1, U4.GND@2, U4.GND@3, U5./OE1, U5./OE2, U5.A8, U7.DISABLE, U7.GND
- net GO: now also U7.GOUT; no longer U2.GOUT
- net MODE: now also U7.NT/PAL; no longer U2.NT/PAL
- net N$10: now also C29.2, U7.RCLAMP; no longer C6.2, U2.RCLAMP
- net N$11: now also C30.2, U7.GCLAMP; no longer C26.2, U2.GCLAMP
- net N$12: now also C31.2, U7.BCLAMP; no longer C27.2, U2.BCLAMP
- net N$13: now also C32.2, U7.VREFOUT; no longer C28.2, U2.VREFOUT
- net N$14: now also C24.2; no longer C30.2
- net N$15: now also U6.BYPASS; no longer U7.BYPASS
- net N$16: now also C25.2; no longer C31.2
- net N$17: now also C23.1, U6.CH4_IN; no longer C29.1, U7.CH4_IN
- net N$18: now also C24.1, U6.CH3_IN; no longer C30.1, U7.CH3_IN
- net N$19: now also C25.1, U6.CH2_IN; no longer C31.1, U7.CH2_IN
- net N$2: now also U5.Y; no longer U6.Y
- net N$20: now also C26.2; no longer C32.2
- net N$21: now also C26.1, U6.CH1_IN; no longer C32.1, U7.CH1_IN
- net N$22: now also U2.A2; no longer U3.A2
- net N$23: now also U2.A3; no longer U3.A3
- net N$24: now also U4.A6; no longer U5.A6
- net N$25: now also U2.A4; no longer U3.A4
- net N$26: now also U2.A5; no longer U3.A5
- net N$27: now also U2.A6; no longer U3.A6
- net N$28: now also U2.A7; no longer U3.A7
- net N$29: now also U7.YTRAP; no longer U2.YTRAP
- net N$3: now also U4.A5; no longer U5.A5
- net N$30: now also C35.2; no longer C36.2
- net N$31: now also U7.COUT; no longer U2.COUT
- net N$32: now also U7.VOUT; no longer U2.VOUT
- net N$33: now also C33.2; no longer C37.2
- net N$34: now also C34.2; no longer C38.2
- net N$37: now also U7.SCIN; no longer U2.SCIN
- net N$42: now also C23.2; no longer C29.2
- net N$6: now also U7.VCLK; no longer U2.VCLK
- net N$64: now also U6.CH1_OUT; no longer U7.CH1_OUT
- net N$65: now also U6.CH2_OUT; no longer U7.CH2_OUT
- net N$66: now also U6.CH3_OUT; no longer U7.CH3_OUT
- net N$67: now also U6.CH4_OUT; no longer U7.CH4_OUT
- net N$8: now also U2.A0; no longer U3.A0
- net N$9: now also U2.A1; no longer U3.A1
- net PD0: now also U2.B0; no longer U3.B0
- net PD1: now also U2.B1; no longer U3.B1
- net PD2: now also U2.B2; no longer U3.B2
- net PD3: now also U2.B3; no longer U3.B3
- net PD4: now also U2.B4; no longer U3.B4
- net PD5: now also U2.B5; no longer U3.B5
- net PD6: now also U2.B6; no longer U3.B6
- net PD7: now also U2.B7; no longer U3.B7
- net R/W: now also U4.A7; no longer U5.A7
- net R0: now also U7.R0; no longer U2.R0
- net R1: now also U7.R1; no longer U2.R1
- net R2: now also U7.R2; no longer U2.R2
- net R3: now also U7.R3; no longer U2.R3
- net R4: now also U7.R4; no longer U2.R4
- net R5: now also U7.R5; no longer U2.R5
- net R6: now also U7.R6; no longer U2.R6
- net R7: now also U7.R7; no longer U2.R7
- net RO: now also U7.ROUT; no longer U2.ROUT
- net RW_FPGA: now also U3.DIR, U4.Y7; no longer U4.DIR, U5.Y7
- net SYNCIN: now also U7.SYNCIN; no longer U2.SYNCIN
- net V: now also C34.1; no longer C38.1
- net VCCIO: now also C12.1, C13.2, C17.1, C18.2, C19.1, U2.VCCA, U4.VCC; no longer C13.1, C17.2, C18.1, C19.2, C23.1, U4.VCCA, U6.VCC
- net VR10_FPGA: now also U4.Y5; no longer U5.Y5
- net VRCS_FPGA: now also U4.Y6; no longer U5.Y6
- net YO: now also U7.YOUT; no longer U2.YOUT
Other:
- moved on the sheet: C1, C11, C12, C13, C14, C15, C16, C17, C18, C19, C2, C20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

Commit message: Add files via upload
Parts:
- R1: value 100 -> 1к
Changed lines of the file:
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@@
 <?xml version="1.0" encoding="utf-8"?>
 <!DOCTYPE eagle SYSTEM "eagle.dtd">
-<eagle version="9.6.2">
+<eagle version="9.4.2">
 <drawing>
 <settings>
@@
 <setting verticaltext="up"/>
 </settings>
-<grid distance="0.1" unitdist="inch" unit="inch" style="lines" multiple="1" display="yes" altdistance="0.01" altunitdist="inch" altunit="inch"/>
+<grid distance="0.1" unitdist="inch" unit="inch" style="lines" multiple="1" display="no" altdistance="0.01" altunitdist="inch" altunit="inch"/>
 <layers>
 <layer number="1" name="Top" color="4" fill="1" visible="no" active="no"/>
@@
 <part name="T1" library="transistor" library_urn="urn:adsk.eagle:library:402" deviceset="BC847" device="" package3d_urn="urn:adsk.eagle:package:28738/2"/>
 <part name="GND1" library="supply1" library_urn="urn:adsk.eagle:library:371" deviceset="GND" device=""/>
-<part name="R1" library="rcl" library_urn="urn:adsk.eagle:library:334" deviceset="R-EU_" device="R0805" package3d_urn="urn:adsk.eagle:package:23553/2" value="100"/>
+<part name="R1" library="rcl" library_urn="urn:adsk.eagle:library:334" deviceset="R-EU_" device="R0805" package3d_urn="urn:adsk.eagle:package:23553/2" value="1к"/>
 <part name="J2" library="jumper" library_urn="urn:adsk.eagle:library:252" deviceset="JP1E" device="" package3d_urn="urn:adsk.eagle:package:15455/1" value="DENDY"/>
 <part name="J3" library="jumper" library_urn="urn:adsk.eagle:library:252" deviceset="JP1E" device="" package3d_urn="urn:adsk.eagle:package:15455/1" value="PALSEL0"/>
