File: PCB Cyclone I/PCB V2.1/PPU_LITE.sch (EAGLE design)
At the start: 91 parts, among them CON1 DIP40, J1 NTSC/PAL, J2 DENDY, J3 PALSEL0, J4 PALSEL1, J5 PIN1-2, J6 PIN1-2, J9 BYPASS, T1 BC847, U1 EP1C3T100C8N, U2 EPCS4, U3 SN74LVC8T245, U4 SN74LVC8T245, U5 SN74LVC541A, U7 THS7374IPWR, X1 057-010-1

Commit message: Add files via upload
Parts:
- removed J5, J6: PIN1-2, con-faston:PIN1-2
- removed R28, R29, R30: 1k, rcl:R-EU_R0805
- removed R31: 100k, rcl:R-EU_R0805
- added C5: 22uF, rcl_my:C-EUC0603
- L1: value BLM31 -> (none)
Connections:
- net +3V3: now also C5.2; no longer R29.1, R30.1
- net ASDO: now also U2.ASDI; no longer U2.DATA
- net DATA0: now also U2.DATA; no longer U2.ASDI
- net GND: no longer R28.1, R31.2
- net N$13: no longer R31.1
- net TCK: no longer R28.2
- net TDI: no longer R29.2
- net TMS: no longer R30.2
- net VRAMA10: no longer J6.1
- net VRAMCS: no longer J5.1
Other:
- moved on the sheet: X1-1, X1-10, X1-2, X1-3, X1-4, X1-5, X1-6, X1-7, X1-8, X1-9

Commit message: Add files via upload
Connections:
- removed net +3V3: C10.1, C12.1, C19.1, C20.1, C21.1, C24.1, C25.1, C26.2, C27.2, C28.2, C29.2, C3.2, C30.1, C4.2, C5.2, C6.2, C9.2, R3.1, R5.2, R6.2, U1.VCC_IO1@1, U1.VCC_IO2@1, U1.VCC_IO2@2, U1.VCC_IO3, U1.VCC_IO4@1, U1.VCC_IO4@2, U2.VCC@1, U2.VCC@2, U2.VCC@3, U3.VCCA, U4.VCCA, U5.VCC, VR1.VOUT, VR2.VIN, X1-4.S, XO1.VDD
- new net N$3: C6.2, VR2.VIN
- new net VCCIO: C10.1, C12.1, C19.1, C20.1, C21.1, C24.1, C25.1, C26.2, C27.2, C28.2, C29.2, C3.2, C30.1, C4.2, C5.2, C9.2, R3.1, R5.2, R6.2, U1.VCC_IO1@1, U1.VCC_IO2@1, U1.VCC_IO2@2, U1.VCC_IO3, U1.VCC_IO4@1, U1.VCC_IO4@2, U2.VCC@1, U2.VCC@2, U2.VCC@3, U3.VCCA, U4.VCCA, U5.VCC, VR1.VOUT, X1-4.S, XO1.VDD
- net GND: now also C1.1, C10.2, C11.1, C12.2, C13.1, C14.1, C15.1, C16.1, C17.1, C18.1, C19.2, C2.1, C20.2, C21.2, C22.1, C23.1, C24.2, C25.2, C26.1, C27.1, C3.1, C30.2, C31.1, C4.1, C5.1, C6.1, C7.1, C8.1, C9.1, VR1.GND, VR2.GND
Other:
- moved on the sheet: C6, C7, C8, C9, U5, VR2, X1-1, X1-3, X1-5, X1-7, X1-9

Commit message: Add files via upload
Parts:
- added JP1: VRAMCS, pinhead:PINHD-1X1
- added JP3: VRAMA10, pinhead:PINHD-1X1
Connections:
- removed net VRAMA10: U5.A7
- removed net VRAMCS: U5.A1
- new net N$18: JP1.1, U5.A1
- new net N$19: JP3.1, U5.A7

Commit message: Add files via upload
Parts:
- JP2: value (none) -> AVOUT
- L1: value (none) -> BLM31
Connections:
- removed net N$3: C6.2, VR2.VIN
- removed net N$33: RN4A.1, RN4B.1, RN4D.2, RN6A.2
- removed net N$36: RN5B.2, RN6B.1, RN6C.2
- removed net N$37: RN5C.2, RN6C.1, RN6D.2
- new net N$25: RN4A.1, RN6A.2, RN6B.1
- new net N$26: RN5A.2, RN5B.2, RN5C.1
- new net N$28: RN5A.1, RN5B.1, RN5D.1, RN6A.1
- net +5V: now also C11.1, C13.1; no longer C11.2, C13.2
- net B0: now also RN8C.2; no longer RN7C.1
- net B1: now also RN8D.2; no longer RN7D.1
- net B2: now also RN7A.2; no longer RN8A.1
- net B3: now also RN7B.2; no longer RN8B.1
- net B4: now also RN7C.2; no longer RN8C.1
- net B5: now also RN7D.2; no longer RN8D.1
- net G0: now also RN5C.2; no longer RN4C.1
- net G1: now also RN5D.2; no longer RN4D.1
- net G2: now also RN4A.2; no longer RN5A.1
- net G3: now also RN4B.2; no longer RN5B.1
- net G4: now also RN4C.2; no longer RN5C.1
- net G5: now also RN4D.2; no longer RN5D.1
- net GND: now also C11.2, C13.2; no longer C11.1, C13.1
- net N$17: now also RN7A.1, RN9A.2, RN9B.1; no longer RN8A.2, RN9A.1, RN9B.2
- net N$21: now also RN8A.2, RN8B.2, RN8C.1; no longer RN7A.2, RN7B.2, RN7C.2
- net N$22: now also RN8A.1, RN8B.1, RN8D.1, RN9A.1; no longer RN7A.1, RN7B.1, RN7D.2, RN9A.2
- net N$23: now also RN7B.1, RN9B.2, RN9C.1; no longer RN8B.2, RN9B.1, RN9C.2
- net N$27: now also RN7C.1, RN9C.2, RN9D.1; no longer RN8C.2, RN9C.1, RN9D.2
- net N$29: now also RN7D.1, RN9D.2; no longer RN8D.2, RN9D.1
- net N$31: now also RN4B.1, RN6C.1; no longer RN5A.2, RN6A.1
- net N$32: now also RN4C.1, RN6C.2, RN6D.1; no longer RN4A.2, RN4B.2, RN4C.2
- net N$38: now also RN4D.1, RN6D.2; no longer RN5D.2, RN6D.1
- net N$45: now also RN1A.1, RN3A.2, RN3B.1; no longer RN2A.2, RN3A.1, RN3B.2
- net N$46: now also RN2A.2, RN2B.2, RN2C.1; no longer RN1A.2, RN1B.2, RN1C.2
- net N$47: now also RN2A.1, RN2B.1, RN2D.1, RN3A.1; no longer RN1A.1, RN1B.1, RN1D.2, RN3A.2
- net N$50: now also RN1B.1, RN3B.2, RN3C.1; no longer RN2B.2, RN3B.1, RN3C.2
- net N$51: now also RN1C.1, RN3C.2, RN3D.1; no longer RN2C.2, RN3C.1, RN3D.2
- net N$52: now also RN1D.1, RN3D.2; no longer RN2D.2, RN3D.1
- net R0: now also RN2C.2; no longer RN1C.1
- net R1: now also RN2D.2; no longer RN1D.1
- net R2: now also RN1A.2; no longer RN2A.1
- net R3: now also RN1B.2; no longer RN2B.1
- net R4: now also RN1C.2; no longer RN2C.1
- net R5: now also RN1D.2; no longer RN2D.1
- net VCCIO: now also C6.2, VR2.VIN
Other:
- moved on the sheet: C1, C10, C11, C12, C13, C18, C2, C24, C3, C4, C5, C6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

Commit message: Add files via upload
Parts:
- R2: value 100 -> 1k
Changed lines of the file:
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@@
 <?xml version="1.0" encoding="utf-8"?>
 <!DOCTYPE eagle SYSTEM "eagle.dtd">
-<eagle version="9.6.2">
+<eagle version="9.4.2">
 <drawing>
 <settings>
@@
 <setting verticaltext="up"/>
 </settings>
-<grid distance="0.1" unitdist="inch" unit="inch" style="lines" multiple="1" display="yes" altdistance="0.01" altunitdist="inch" altunit="inch"/>
+<grid distance="0.1" unitdist="inch" unit="inch" style="lines" multiple="1" display="no" altdistance="0.01" altunitdist="inch" altunit="inch"/>
 <layers>
 <layer number="1" name="Top" color="4" fill="1" visible="no" active="no"/>
@@
 <part name="T1" library="transistor" library_urn="urn:adsk.eagle:library:402" deviceset="BC847" device="" package3d_urn="urn:adsk.eagle:package:28738/2"/>
 <part name="GND1" library="supply1" library_urn="urn:adsk.eagle:library:371" deviceset="GND" device=""/>
-<part name="R2" library="rcl" library_urn="urn:adsk.eagle:library:334" deviceset="R-EU_" device="R0805" package3d_urn="urn:adsk.eagle:package:23553/2" value="100"/>
+<part name="R2" library="rcl" library_urn="urn:adsk.eagle:library:334" deviceset="R-EU_" device="R0805" package3d_urn="urn:adsk.eagle:package:23553/2" value="1k"/>
 <part name="J2" library="jumper" library_urn="urn:adsk.eagle:library:252" deviceset="JP1E" device="" package3d_urn="urn:adsk.eagle:package:15455/1" value="DENDY"/>
 <part name="J3" library="jumper" library_urn="urn:adsk.eagle:library:252" deviceset="JP1E" device="" package3d_urn="urn:adsk.eagle:package:15455/1" value="PALSEL0"/>
